File: pcb/power_supply_hat/power_supply_hat.kicad_pcb (KiCad board)
At the start: 2 copper layers, 65 x 56 mm, 32 parts, among them J1 GPIO, J2 12v, J3 IMU, Q1 2STD1665, U2 BD9G341EFJ

Commit message: updated pcb
Parts:
- R8: value 1k -> 100k
- moved C5 4.84 mm to (139.1, 62.5)
Connections:
- D1 pad 3: Net-(D1-K) -> (no net)
- D3 pad 3: (no net) -> +5V
Routing:
- net GND: track 144.7 -> 150.2 mm
- net +5V: track 64.1 -> 68.6 mm
- net Net-(D3-A): track 40.0 -> 44.3 mm
Changed lines of the file:
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@@
 			(drillshape 0)
 			(scaleselection 1)
-			(outputdirectory "power_supply_hat_gerber")
+			(outputdirectory "power_supply_hat_gerber/")
 		)
 	)
@@
 			)
 		)
-		(property "Value" "1k"
+		(property "Value" "100k"
 			(at 0 1.17 0)
 			(layer "F.Fab")
@@
 			(layers "F.Cu" "F.Mask" "F.Paste")
 			(roundrect_rratio 0.208333)
-			(net 35 "Net-(D1-K)")
 		)
 		(embedded_fonts no)
@@
 			(layers "F.Cu" "F.Mask" "F.Paste")
 			(roundrect_rratio 0.208333)
+			(net 30 "+5V")
 		)
 		(embedded_fonts no)
@@
 	(footprint "Capacitor_SMD:C_1206_3216Metric_Pad1.33x1.80mm_HandSolder"
 		(layer "F.Cu")
-		(at 136.45 66.575)
+		(at 139.0625 62.5)
 		(descr "Capacitor SMD 1206 (3216 Metric), square (rectangular) end terminal, IPC-7351 nominal with elongated pad for handsoldering. (Body size source: IPC-SM-782 page 76, https://www.pcb-3d.com/wordpress/wp-content/uploads/ipc-sm-782a_amendment_1_and_2.pdf), generated with kicad-footprint-generator")
 		(tags "capacitor handsolder")
@@
 	)
 	(segment
+		(start 140.625 71.475)
+		(end 140.625 62.5)
+		(width 1)
+		(layer "F.Cu")
+		(net 1)
+	)
+	(segment
 		(start 137.8375 83.1875)
 		(end 137.45 83.575)
@@
 	)
 	(segment
+		(start 137.2 74.4)
+		(end 137.45 74.65)
+		(width 1)
+		(layer "F.Cu")
+		(net 1)
+	)
+	(segment
 		(start 107 54.5)
 		(end 105 54.5)
@@
 	)
 	(segment
-		(start 137.45 67.1375)
-		(end 138.0125 66.575)
+		(start 109 55.0625)
+		(end 107.5625 55.0625)
 		(width 1.4)
 		(layer "F.Cu")
@@
 	)
 	(segment
-		(start 109 55.0625)
-		(end 107.5625 55.0625)
-		(width 1.4)
+		(start 137.45 74.65)
+		(end 137.45 83.575)
+		(width 1)
 		(layer "F.Cu")
 		(net 1)
@@
 		(start 113.8 75.6)
 		(end 113.8 71.8)
-		(width 1.4)
+		(width 1)
 		(layer "F.Cu")
 		(net 1)
 	)
 	(segment
-		(start 137.45 83.575)
-		(end 137.45 67.1375)
-		(width 1.4)
+		(start 137.45 74.65)
+		(end 140.625 71.475)
+		(width 1)
 		(layer "F.Cu")
 		(net 1)
@@
 		(start 113.8 71.8)
 		(end 113.9 71.7)
-		(width 1.4)
+		(width 1)
 		(layer "F.Cu")
 		(net 1)
@@
 		(start 103.86 85.54)
 		(end 113.8 75.6)
-		(width 1.4)
+		(width 1)
 		(layer "B.Cu")
 		(net 1)
@@
 		(start 102.5 85.54)
 		(end 103.86 85.54)
-		(width 1.4)
+		(width 1)
 		(layer "B.Cu")
 		(net 1)
@@
 	)
 	(segment
+		(start 133.305 54.775)
+		(end 128.745 54.775)
+		(width 1.4)
+		(layer "F.Cu")
+		(net 30)
+	)
+	(segment
 		(start 109 51.9375)
 		(end 107.1625 51.9375)
@@
 	)
 	(segment
-		(start 134.8875 66.575)
-		(end 131.025 66.575)
-		(width 1.4)
-		(layer "F.Cu")
-		(net 41)
-	)
-	(segment
 		(start 128.95 94.95)
 		(end 128.75 94.75)
@@
 		(layer "F.Cu")
 		(net 41)
+	)
+	(segment
+		(start 131.025 66.575)
+		(end 135.1 62.5)
+		(width 1)
+		(layer "F.Cu")
+		(net 41)
+	)
+	(segment
+		(start 135.1 62.5)
+		(end 137.5 62.5)
+		(width 1)
+		(layer "F.Cu")
+		(net 41)
